File: flatsat-backplane-breakout-debug/flatsat-backplane-breakout-debug/flatsat-backplane-breakout-debug.kicad_pcb (KiCad board)
At the start: 2 copper layers, 1 part

Commit message: Test commit 2
Parts:
- added REF**: BatteryHolder_Keystone_107_1x23mm, Battery:BatteryHolder_Keystone_107_1x23mm, F.Cu at (177.8, 94.0)
Changed lines of the file:
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@@
+    )
+  )
+  (footprint "Battery:BatteryHolder_Keystone_107_1x23mm" (layer "F.Cu")
+    (at 177.8 93.98)
+    (descr "http://www.keyelco.com/product-pdf.cfm?p=746")
+    (tags "Keystone type 107 battery holder")
+    (attr through_hole)
+    (fp_text reference "REF**" (at -1.25 -4.5) (layer "F.SilkS")
+        (effects (font (size 1 1) (thickness 0.15)))
+    )
+    (fp_text value "BatteryHolder_Keystone_107_1x23mm" (at 15 15) (layer "F.Fab")
+        (effects (font (size 1 1) (thickness 0.15)))
+    )
+    (fp_text user "+" (at 2.75 0) (layer "F.SilkS")
+        (effects (font (size 1.5 1.5) (thickness 0.15)))
+    )
+    (fp_text user "${REFERENCE}" (at 7.1 -3.15) (layer "F.Fab")
+        (effects (font (size 1 1) (thickness 0.15)))
+    )
+    (fp_line (start -2.05 -2.5) (end -2.05 2.5)
+      (stroke (width 0.12) (type solid)) (layer "F.SilkS"))
+    (fp_line (start -1.5 3.05) (end 0.95 3.05)
+      (stroke (width 0.12) (type solid)) (layer "F.SilkS"))
+    (fp_line (start 0.95 -3.05) (end -1.5 -3.05)
+      (stroke (width 0.12) (type solid)) (layer "F.SilkS"))
+    (fp_arc (start -2.05 -2.5) (mid -1.888909 -2.888909) (end -1.5 -3.05)
+      (stroke (width 0.12) (type solid)) (layer "F.SilkS"))
+    (fp_arc (start -1.5 3.05) (mid -1.888909 2.888909) (end -2.05 2.5)
+      (stroke (width 0.12) (type solid)) (layer "F.SilkS"))
+    (fp_arc (start 0.95 3.05) (mid 1.371574 3.1784) (end 1.65 3.52)
+      (stroke (width 0.12) (type solid)) (layer "F.SilkS"))
+    (fp_arc (start 1.65 -3.604769) (mid 17.016593 -13.966381) (end 29.2 0)
+      (stroke (width 0.12) (type solid)) (layer "F.SilkS"))
+    (fp_arc (start 1.65 -3.52) (mid 1.371575 -3.1784) (end 0.95 -3.05)
+      (stroke (width 0.12) (type solid)) (layer "F.SilkS"))
+    (fp_arc (start 29.2 0) (mid 16.974433 13.886952) (end 1.65 3.52)
+      (stroke (width 0.12) (type solid)) (layer "F.SilkS"))
+    (fp_line (start -2.3 -2.5) (end -2.3 2.5)
+      (stroke (width 0.05) (type solid)) (layer "F.CrtYd"))
+    (fp_line (start -1.5 3.3) (end 0.95 3.3)
+      (stroke (width 0.05) (type solid)) (layer "F.CrtYd"))
+    (fp_line (start 0.95 -3.3) (end -1.5 -3.3)
+      (stroke (width 0.05) (type solid)) (layer "F.CrtYd"))
+    (fp_arc (start -2.3 -2.5) (mid -2.065685 -3.065685) (end -1.5 -3.3)
+      (stroke (width 0.05) (type solid)) (layer "F.CrtYd"))
+    (fp_arc (start -1.5 3.3) (mid -2.065685 3.065685) (end -2.3 2.5)
+      (stroke (width 0.05) (type solid)) (layer "F.CrtYd"))
+    (fp_arc (start 0.95 3.3) (mid 1.22459 3.381628) (end 1.41 3.6)
+      (stroke (width 0.05) (type solid)) (layer "F.CrtYd"))
+    (fp_arc (start 1.41 -3.6) (mid 1.224591 -3.381627) (end 0.95 -3.3)
+      (stroke (width 0.05) (type solid)) (layer "F.CrtYd"))
+    (fp_arc (start 1.41 -3.6) (mid 17.014123 -14.138563) (end 29.45 0)
+      (stroke (width 0.05) (type solid)) (layer "F.CrtYd"))
+    (fp_arc (start 29.45 0) (mid 17.014124 14.138563) (end 1.41 3.6)
+      (stroke (width 0.05) (type solid)) (layer "F.CrtYd"))
+    (fp_line (start -1.9 -2.5) (end -1.9 2.5)
+      (stroke (width 0.1) (type solid)) (layer "F.Fab"))
+    (fp_line (start -1.5 2.9) (end 0.95 2.9)
+      (stroke (width 0.1) (type solid)) (layer "F.Fab"))
+    (fp_line (start 0 -1.3) (end 0 1.3)
+      (stroke (width 0.1) (type solid)) (layer "F.Fab"))
+    (fp_line (start 0 1.3) (end 16.2 1.3)
+      (stroke (width 0.1) (type solid)) (layer "F.Fab"))
+    (fp_line (start 0.95 -2.9) (end -1.5 -2.9)
+      (stroke (width 0.1) (type solid)) (layer "F.Fab"))
+    (fp_line (start 16.2 -1.3) (end 0 -1.3)
+      (stroke (width 0.1) (type solid)) (layer "F.Fab"))
+    (fp_line (start 23.7109 -7.8867) (end 25.3392 -9.4388)
+      (stroke (width 0.1) (type solid)) (layer "F.Fab"))
+    (fp_line (start 23.7236 7.8613) (end 25.3673 9.3907)
+      (stroke (width 0.1) (type solid)) (layer "F.Fab"))
+    (fp_arc (start -1.9 -2.5) (mid -1.782843 -2.782843) (end -1.5 -2.9)
+      (stroke (width 0.1) (type solid)) (layer "F.Fab"))
+    (fp_arc (start -1.5 2.9) (mid -1.782843 2.782843) (end -1.9 2.5)
+      (stroke (width 0.1) (type solid)) (layer "F.Fab"))
+    (fp_arc (start 0.95 2.9) (mid 1.470216 3.06511) (end 1.8 3.5)
+      (stroke (width 0.1) (type solid)) (layer "F.Fab"))
+    (fp_arc (start 1.8 -3.5) (mid 1.470217 -3.06511) (end 0.95 -2.9)
+      (stroke (width 0.1) (type solid)) (layer "F.Fab"))
+    (fp_arc (start 1.8 -3.5) (mid 16.964356 -13.736686) (end 29.049508 0)
+      (stroke (width 0.1) (type solid)) (layer "F.Fab"))
+    (fp_arc (start 3.7 -1.3) (mid 16.5 -11.5) (end 26.7 1.3)
+      (stroke (width 0.1) (type solid)) (layer "F.Fab"))
+    (fp_arc (start 9 -1.3) (mid 15.851289 -6.300938) (end 21.53 0)
+      (stroke (width 0.1) (type solid)) (layer "F.Fab"))
+    (fp_arc (start 13.3 -1.3) (mid 15.963947 -2.171724) (end 17.495448 0.175833)
+      (stroke (width 0.1) (type solid)) (layer "F.Fab"))
+    (fp_arc (start 16.2 -1.3) (mid 17.5 0) (end 16.2 1.3)
+      (stroke (width 0.1) (type solid)) (layer "F.Fab"))
+    (fp_arc (start 17.495448 -0.175833) (mid 15.963947 2.171724) (end 13.3 1.3)
+      (stroke (width 0.1) (type solid)) (layer "F.Fab"))
+    (fp_arc (start 21.53 0) (mid 15.851292 6.300937) (end 9 1.3)
+      (stroke (width 0.1) (type solid)) (layer "F.Fab"))
+    (fp_arc (start 26.7 -1.3) (mid 16.5 11.5) (end 3.7 1.3)
+      (stroke (width 0.1) (type solid)) (layer "F.Fab"))
+    (fp_arc (start 29.049508 0) (mid 16.964356 13.736685) (end 1.8 3.5)
+      (stroke (width 0.1) (type solid)) (layer "F.Fab"))
+    (pad "1" thru_hole rect (at 0 0) (size 3 3) (drill 1.5) (layers "*.Cu" "*.Mask"))
+    (pad "2" thru_hole circle (at 20.49 0) (size 3 3) (drill 1.5) (layers "*.Cu" "*.Mask"))
+    (model "${KICAD6_3DMODEL_DIR}/Battery.3dshapes/BatteryHolder_Keystone_107_1x23mm.wrl"
+      (offset (xyz 0 0 0))
+      (scale (xyz 1 1 1))
+      (rotate (xyz 0 0 0))
     )
   )
