File: backplane-debug-breakout/backplane-debug-breakout.kicad_pcb (KiCad board)
At the start: 2 copper layers, 60 x 63 mm, 21 parts, among them J1 Conn_02x08_Odd_Even, J2 Conn_01x04, J4 Conn_01x02_Socket, J5 Conn_01x04, J6 629105150521, SW1 SW_Push_DPDT, SW2 SW_Omron_B3FS, SW3 EG1218, U1 UMFT234XF

Commit message: Changes generic values on switches to mfgr part number. Re-ran ERC and DRC, made vulcan adapter to be PCB only, and updated to 8.0.7.
Parts:
- R1: value R_US -> 4.7k
- SW1: value SW_Push_DPDT -> EG2209
- SW2: value SW_Omron_B3FS -> B3F-1000
Changed lines of the file:
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@@
 			)
 		)
-		(property "Value" "SW_Omron_B3FS"
+		(property "Value" "B3F-1000"
 			(at 2.9 -2.5 180)
 			(layer "F.Fab")
@@
 			)
 		)
-		(attr exclude_from_pos_files exclude_from_bom)
+		(attr board_only exclude_from_pos_files exclude_from_bom)
 		(fp_rect
 			(start -3.175 -3.175)
@@
 			)
 		)
-		(property "Value" "SW_Push_DPDT"
+		(property "Value" "EG2209"
 			(at 0.2 -6.6 90)
 			(layer "F.SilkS")
@@
 			)
 		)
+		(property "DPN" "EG1907-ND"
+			(at 0 0 -90)
+			(unlocked yes)
+			(layer "F.Fab")
+			(hide yes)
+			(effects
+				(font
+					(size 1 1)
+					(thickness 0.15)
+				)
+			)
+		)
+		(property "DST" "Digi-Key"
+			(at 0 0 -90)
+			(unlocked yes)
+			(layer "F.Fab")
+			(hide yes)
+			(effects
+				(font
+					(size 1 1)
+					(thickness 0.15)
+				)
+			)
+		)
+		(property "MFR" "E-Switch"
+			(at 0 0 -90)
+			(unlocked yes)
+			(layer "F.Fab")
+			(hide yes)
+			(effects
+				(font
+					(size 1 1)
+					(thickness 0.15)
+				)
+			)
+		)
+		(property "MPN" "EG2209"
+			(at 0 0 -90)
+			(unlocked yes)
+			(layer "F.Fab")
+			(hide yes)
+			(effects
+				(font
+					(size 1 1)
+					(thickness 0.15)
+				)
+			)
+		)
 		(sheetname "Root")
 		(sheetfile "backplane-debug-breakout.kicad_sch")
@@
 			)
 		)
-		(property "Value" "R_US"
+		(property "Value" "4.7k"
 			(at 0 1.43 180)
 			(layer "F.Fab")
@@
 			)
 		)
+		(property "DPN" "RMCF0603FT4K70CT-ND"
+			(at 0 0 180)
+			(unlocked yes)
+			(layer "F.Fab")
+			(hide yes)
+			(effects
+				(font
+					(size 1 1)
+					(thickness 0.15)
+				)
+			)
+		)
+		(property "DST" "Digi-Key"
+			(at 0 0 180)
+			(unlocked yes)
+			(layer "F.Fab")
+			(hide yes)
+			(effects
+				(font
+					(size 1 1)
+					(thickness 0.15)
+				)
+			)
+		)
+		(property "MFR" "Stackpole Electronics Inc"
+			(at 0 0 180)
+			(unlocked yes)
+			(layer "F.Fab")
+			(hide yes)
+			(effects
+				(font
+					(size 1 1)
+					(thickness 0.15)
+				)
+			)
+		)
+		(property "MPN" "RMCF0603FT4K70"
+			(at 0 0 180)
+			(unlocked yes)
+			(layer "F.Fab")
+			(hide yes)
+			(effects
+				(font
+					(size 1 1)
+					(thickness 0.15)
+				)
+			)
+		)
 		(property ki_fp_filters "R_*")
 		(sheetname "Root")
@@
 			)
 		)
+		(property "DPN" "587-3472-1-ND"
+			(at 0 0 180)
+			(unlocked yes)
+			(layer "F.Fab")
+			(hide yes)
+			(effects
+				(font
+					(size 1 1)
+					(thickness 0.15)
+				)
+			)
+		)
+		(property "DST" "Digi-Key"
+			(at 0 0 180)
+			(unlocked yes)
+			(layer "F.Fab")
+			(hide yes)
+			(effects
+				(font
+					(size 1 1)
+					(thickness 0.15)
+				)
+			)
+		)
+		(property "MFR" "Taiyo Yuden"
+			(at 0 0 180)
+			(unlocked yes)
+			(layer "F.Fab")
+			(hide yes)
+			(effects
+				(font
+					(size 1 1)
+					(thickness 0.15)
+				)
+			)
+		)
+		(property "MPN" "TMK107BJ104KAHT"
+			(at 0 0 180)
+			(unlocked yes)
+			(layer "F.Fab")
+			(hide yes)
+			(effects
+				(font
+					(size 1 1)
+					(thickness 0.15)
+				)
+			)
+		)
 		(property ki_fp_filters "C_*")
 		(sheetname "Root")
@@
 					(thickness 0.15)
 				)
+			)
+		)
+		(property "DPN" "732-4978-1-ND"
+			(at 0 0 0)
+			(unlocked yes)
+			(layer "F.Fab")
+			(hide yes)
+			(effects
+				(font
+					(size 1 1)
+					(thickness 0.15)
+				)
+			)
+		)
+		(property "DST" "Digi-Key"
+			(at 0 0 0)
+			(unlocked yes)
+			(layer "F.Fab")
+			(hide yes)
+			(effects
+				(font
+					(size 1 1)
+					(thickness 0.15)
+				)
+			)
+		)
+		(property "MFR" "Wurth"
+			(at 0 0 0)
+			(unlocked yes)
+			(layer "F.Fab")
+			(hide yes)
+			(effects
+				(font
+					(size 1 1)
+					(thickness 0.15)
+				)
+			)
+		)
+		(property "MPN" "150060RS75000"
+			(at 0 0 0)
+			(unlocked yes)
+			(layer "F.Fab")
+			(hide yes)
+			(effects
+				(font
+					(size 1 1)
+					(thickness 0.15)
+				)
