File: c3-surrogate-card/oresat-c3-surrogate.kicad_pcb (KiCad board)
At the start: 2 copper layers, 99.8 x 94.6 mm, 73 parts, among them J1 J-SAMTEC-TFM-120-X1-XXX-D-RA, J2 Conn_01x04, J4 1995499, Q1 PMV45EN, Q3 NTR4101P, Q4 NTR4101P, Q5 DMP3050LVT-7, SW2 EG1218, SW3 OS203011MV9QS1, SW4 EG1218, U1 MAX892LEUA+T, U2 LTC4412xS6, U4 LTC4412xS6, U5 TS5A21366

Commit message: Updated Trinket M0 symbol to be sane and update with pinout picture.
Connections:
- net Net-(PCB3-SCL) renamed /SCL
- net Net-(PCB3-SDA) renamed /SDA
Changed lines of the file:
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@@
 	(net 50 "Net-(R8-Pad2)")
 	(net 51 "Net-(R9-Pad2)")
-	(net 52 "Net-(PCB3-SDA)")
+	(net 52 "/SDA")
 	(net 53 "unconnected-(PCB3-VBAT-Pad1)")
 	(net 54 "unconnected-(SW3-Pad8)")
@@
 	(net 61 "Net-(U4-CTL)")
 	(net 62 "unconnected-(PCB3-VUSB-Pad10)")
-	(net 63 "Net-(PCB3-SCL)")
+	(net 63 "/SCL")
 	(net 64 "unconnected-(PCB3-RST-Pad5)")
 	(net 65 "unconnected-(SW3-Pad1)")
@@
 			(remove_unused_layers no)
 			(net 27 "/OPD_~{FAULT}")
-			(pinfunction "TX")
+			(pinfunction "D4")
 			(pintype "output")
 		)
@@
 			(remove_unused_layers no)
 			(net 28 "/OPD_~{ENABLE}")
-			(pinfunction "RX")
+			(pinfunction "D3")
 			(pintype "input")
 		)
@@
 			(layers "*.Cu" "*.Mask")
 			(remove_unused_layers no)
-			(net 63 "Net-(PCB3-SCL)")
-			(pinfunction "SCL")
+			(net 63 "/SCL")
+			(pinfunction "RX/SCL/D2")
 			(pintype "bidirectional")
 		)
@@
 			(remove_unused_layers no)
 			(net 26 "/OPD_ISET")
-			(pinfunction "Aout")
+			(pinfunction "D1")
 			(pintype "output")
 		)
@@
 			(layers "*.Cu" "*.Mask")
 			(remove_unused_layers no)
-			(net 52 "Net-(PCB3-SDA)")
-			(pinfunction "SDA")
+			(net 52 "/SDA")
+			(pinfunction "TX/SDA/D0")
 			(pintype "bidirectional")
 		)
@@
 			(layers "F.Cu" "F.Mask" "F.Paste")
 			(roundrect_rratio 0.25)
-			(net 63 "Net-(PCB3-SCL)")
+			(net 63 "/SCL")
 			(pintype "passive")
 		)
@@
 			(layers "*.Cu" "*.Mask")
 			(remove_unused_layers no)
-			(net 63 "Net-(PCB3-SCL)")
+			(net 63 "/SCL")
 			(pinfunction "1")
 			(pintype "passive")
@@
 			(layers "F.Cu" "F.Mask" "F.Paste")
 			(roundrect_rratio 0.25)
-			(net 52 "Net-(PCB3-SDA)")
+			(net 52 "/SDA")
 			(pintype "passive")
 		)
@@
 			(layers "F.Cu" "F.Mask" "F.Paste")
 			(roundrect_rratio 0.25)
-			(net 52 "Net-(PCB3-SDA)")
+			(net 52 "/SDA")
 			(pinfunction "COM1")
 			(pintype "passive")
@@
 			(layers "F.Cu" "F.Mask" "F.Paste")
 			(roundrect_rratio 0.25)
-			(net 63 "Net-(PCB3-SCL)")
+			(net 63 "/SCL")
 			(pinfunction "COM2")
 			(pintype "passive")
@@
 			(layers "*.Cu" "*.Mask")
 			(remove_unused_layers no)
-			(net 52 "Net-(PCB3-SDA)")
+			(net 52 "/SDA")
 			(pinfunction "1")
 			(pintype "passive")
