File: card-debug-board-3/card-debug-board-3.kicad_sch (KiCad schematic)
At the start: 101 parts, among them J1 USB4105-GF-A, J2 USB4105-GF-A, J3 Conn_01x05, J4 5040501291, J5 2-1734592-0, Q1 PMV450ENEAR, Q2 PMV450ENEAR, Q3 NTR4101P, SW1 B3F-1000, SW2 PCM13SMTR, SW3 B3F-1000, SW4 SW_DIP_x01, U1 MIC5205-3.3YM5, U2 W25Q16JVSS, U3 RP2040, U4 74AUP1G17, U5 74AUP1G17, U6 IP4234CZ6,125, U7 IP4234CZ6,125, Y1 12 MHz

Commit message: v3.3 of the card debug board, now with automativ solar power control
Parts:
- removed TP20, TP5, TP6: TestPoint-MinTH, oresat-misc:TestPoint-MinTH, symbol oresat-misc:TestPoint-MinTH
- added J6: Conn_01x03, Connector_PinHeader_2.54mm:PinHeader_1x03_P2.54mm_Vertical, symbol Connector_Generic:Conn_01x03
- added Q4: DMP2035UQ-7, Package_TO_SOT_SMD:SOT-23, symbol Transistor_FET:NTR2101P
- added R27: 10k, oresat-passives:0603-C-NOSILK, symbol Device:R_Small_US
- Q1, Q2: value PMV450ENEAR -> DMN3028LQ-7; DPN 1727-2532-1-ND -> 31-DMN3028LQ-7CT-ND; MFR Nexperia -> Diodes Incorporated; MPN PMV450ENEAR -> DMN3028LQ-7
- Q3: value NTR4101P -> DMP2035UQ-7; DPN NTR4101PT1GOSCT-ND -> 31-DMP2035UQ-7CT-ND; MFR ON Semi -> Diodes Incorporated; MPN NTR4101PT1G -> DMP2035UQ-7
Connections:
- net +3.3V: now also Q4.2 (S), R27.2
- net GND: now also J6.3 (Pin_3)
- net TARGET_POWER_SOLAR: now reaches U3.31 (GPIO20)
- net TARGET_POWER_SOLAR: now also Q4.1 (G), R27.1
- net at C1.1: now also J1.SH (SHIELD); no longer J1.S1 (SHIELD)
- net at C2.2: now also J2.SH (SHIELD); no longer J2.S1 (SHIELD)
- net at U3.24 (SWCLK): now also J6.1 (Pin_1)
- net at U3.25 (SWDIO): now also J6.2 (Pin_2)
- net at D7.2 (A), SW4.2: now also Q4.3 (D)
Other:
- note added: "02x JST SHLP-14V-S-B 1.0 mm pitch wire-to-board "SHL" connector And then one set of leads: - 14x JST ASSHLSSHL28K152 28 AWG Jumper Lead Socket to Socket 6.00" (152 mm) - 14x JST ASSHLSSHL28K305 28 AWG Jumper Lead Socket to Socket 12.0" (305 mm) IMPORTANT: Wire pin 1 to pin 1, 2 to 2, etc."
- note added: "PICO SWD"
- note removed: "02x JST SHLP-14V-S-B 1.0 mm pitch wire-to-board "SHL" connector And then one set of leads: - 14x JST ASSHLSSHL28K305 28 AWG Jumper Lead Socket to Socket 12.0" (305 mm) - or - 14x JST ASSHLSSHL28K152 28 AWG Jumper Lead Socket to Socket 6.00" (152 mm) IMPORTANT: CROSS PRECRIMPED WIRES (Wire pin 1 to pin 1!)"
- moved on the sheet: D7, SW4
