File: flatsat-interface-card/flatsat-interface-card.kicad_pcb (KiCad board)
At the start: 2 copper layers, 21 parts, among them J1 J-SAMTEC-TFM-120-01-L-D-RA, J2 J-SAMTEC-TFM-120-01-L-D-RA, U1 MCP2221AxST

Commit message: cleaned up schematic more
Parts:
- removed R1: 10m, Resistor_SMD:R_0805_2012Metric
- added SW1: C&K PCM13SMTR, oresat-misc:SW-CK-PCM13SMTR, F.Cu at (107.7, 92.7)
- added TP18: Test-Point, oresat-misc:TestPoint-0.75mm-th, F.Cu at (155.9, 66.3)
- added TP19: Test-Point, oresat-misc:TestPoint-0.75mm-th, F.Cu at (155.9, 68.9)
- added TP20: Test-Point, oresat-misc:TestPoint-0.75mm-th, F.Cu at (155.9, 71.4)
- added TP21: Test-Point, oresat-misc:TestPoint-0.75mm-th, F.Cu at (155.9, 73.9)
- added TP22: Test-Point, oresat-misc:TestPoint-0.75mm-th, F.Cu at (183.2, 69.7)
- added TP23: Test-Point, oresat-misc:TestPoint-0.75mm-th, F.Cu at (183.2, 72.2)
- added TP24: Test-Point, oresat-misc:TestPoint-0.75mm-th, F.Cu at (165.4, 52.0)
- added TP25: Test-Point, oresat-misc:TestPoint-0.75mm-th, F.Cu at (165.4, 54.5)
- added TP26: Test-Point, oresat-misc:TestPoint-0.75mm-th, F.Cu at (168.0, 52.0)
- added TP27: Test-Point, oresat-misc:TestPoint-0.75mm-th, F.Cu at (168.0, 54.5)
- added TP28: Test-Point, oresat-misc:TestPoint-0.75mm-th, F.Cu at (170.5, 52.0)
- added TP29: Test-Point, oresat-misc:TestPoint-0.75mm-th, F.Cu at (170.5, 54.5)
- added U2: INA226, Package_SO:TSSOP-10_3x3mm_P0.5mm, F.Cu at (140.7, 73.1)
- added U3: LTC4412xS6, Package_TO_SOT_SMD:TSOT-23-6, F.Cu at (159.8, 67.5)
- added U4: LTC4412xS6, Package_TO_SOT_SMD:TSOT-23-6, F.Cu at (159.8, 72.1)
- added U5: TS5A21366, Package_SO:VSSOP-8_2.3x2mm_P0.5mm, F.Cu at (132.9, 69.3)
- added U6: MAX892LEUA+T, oresat-ics:LINEAR-MSOP-8-AND-MAXIM-UMAX-8-21-0036, F.Cu at (134.2, 81.2)
- added U7: MIC23050-SYML, Package_DFN_QFN:Micrel_MLF-8-1EP_2x2mm_P0.5mm_EP0.6x1.2mm_ThermalVias, F.Cu at (126.2, 76.0)
- added U8: LTC4412xS6, Package_TO_SOT_SMD:TSOT-23-6, F.Cu at (179.4, 70.8)
- added U9: IP4234CZ6,125, Package_SO:TSOP-6_1.65x3.05mm_P0.95mm, F.Cu at (164.6, 67.4)
- J1: value J-SAMTEC-TFM-120-01-L-D-RA -> J-SAMTEC-TFM-120-X1-XXX-D-RA
- J2: value J-SAMTEC-TFM-120-01-L-D-RA -> SFM-120-02-X-DH; footprint oresat-connectors:J-SAMTEC-TFM-120-X1-XXX-D-RA -> oresat-connectors:SFM-120-02-X-DH
- moved J1 53.6 mm to (131.2, 103.4), turned to 180 degrees
- moved TP1 34.4 mm to (106.0, 64.5)
- moved TP10 34.4 mm to (108.5, 72.1)
- moved TP11 34.4 mm to (108.5, 74.6)
- moved TP12 34.4 mm to (108.5, 77.1)
- moved TP13 34.4 mm to (111.0, 64.5)
- moved TP14 34.4 mm to (111.0, 67.0)
- moved TP15 34.4 mm to (111.0, 69.5)
- moved TP16 34.4 mm to (111.0, 72.1)
- moved TP17 34.4 mm to (111.0, 74.6)
- moved TP2 34.4 mm to (106.0, 67.0)
- moved TP3 34.4 mm to (106.0, 69.5)
- moved TP4 34.4 mm to (106.0, 72.1)
- moved TP5 34.4 mm to (106.0, 74.6)
- moved TP6 34.4 mm to (106.0, 77.1)
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Connections:
- net /Interfaces/CAN2_H renamed /Bus Interfaces/CAN2_H
- net /Interfaces/CAN2_L renamed /Bus Interfaces/CAN2_L
- net /Interfaces/SPARE1 renamed /Bus Interfaces/SPARE1
- net /Interfaces/SPARE10 renamed /Bus Interfaces/SPARE10
- net /Interfaces/SPARE21 renamed /Bus Interfaces/SPARE21
- net /Interfaces/SPARE22 renamed /Bus Interfaces/SPARE22
- net /Interfaces/SPARE3 renamed /Bus Interfaces/SPARE3
- net /Interfaces/SPARE31 renamed /Bus Interfaces/SPARE31
- net /Interfaces/SPARE32 renamed /Bus Interfaces/SPARE32
- net /Interfaces/SPARE4 renamed /Bus Interfaces/SPARE4
- net /Interfaces/SPARE5 renamed /Bus Interfaces/SPARE5
- net /Interfaces/SPARE6 renamed /Bus Interfaces/SPARE6
- net /Interfaces/SPARE7 renamed /Bus Interfaces/SPARE7
- net /Interfaces/SPARE8 renamed /Bus Interfaces/SPARE8
- net /Interfaces/SPARE9 renamed /Bus Interfaces/SPARE9
- net CAN1_H renamed /Bus Interfaces/CAN1_H
- net CAN1_L renamed /Bus Interfaces/CAN1_L
- net OPD_PWR renamed /Bus Interfaces/OPD_PWR
- net OPD_SCL renamed /Bus Interfaces/OPD_SCL
- net OPD_SDA renamed /Bus Interfaces/OPD_SDA
- net ~{SD} renamed /Bus Interfaces/~{SD}
- J1 pad 37: C3-UART-TX -> /Bus Interfaces/C3-UART-TX
- J1 pad 38: C3-UART-RX -> /Bus Interfaces/C3-UART-RX
- J2 pad 37: C3-UART-TX -> /Bus Interfaces/C3-UART-TX
- J2 pad 38: C3-UART-RX -> /Bus Interfaces/C3-UART-RX
- U1 pad 1: unconnected-(U1-VDD-Pad1) -> VUSB
- U1 pad 10: unconnected-(U1-SCL-Pad10) -> Net-(U1-SCL)
- U1 pad 11: unconnected-(U1-VUSB-Pad11) -> Net-(U1-VUSB)
- U1 pad 12: unconnected-(U1-D--Pad12) -> /Measurement/USB-
- U1 pad 13: unconnected-(U1-D+-Pad13) -> /Measurement/USB+
- U1 pad 14: unconnected-(U1-VSS-Pad14) -> GND
- U1 pad 2: unconnected-(U1-GP0-Pad2) -> /Measurement/USBShutdown
- U1 pad 5: unconnected-(U1-URx-Pad5) -> /Bus Interfaces/C3-UART-TX
- U1 pad 6: unconnected-(U1-UTx-Pad6) -> /Bus Interfaces/C3-UART-RX
- U1 pad 7: unconnected-(U1-GP2-Pad7) -> Net-(Q5-G)
- U1 pad 8: unconnected-(U1-GP3-Pad8) -> Net-(U1-GP3)
- U1 pad 9: unconnected-(U1-SDA-Pad9) -> Net-(U1-SDA)
