File: flatsat-debugger/flatsat-debugger.kicad_sch (KiCad schematic)
At the start: 10 parts, among them J1 J-SAMTEC-TFM-120-X1-XXX-D-RA, J2 SFM-120-02-X-DH, J3 USB_C_Receptacle_USB2.0_16P, J4 Barrel_Jack

Commit message: filename fixes
Other:
- sheet OPD renamed opd
- sheet current sensing: file untitled.kicad_sch -> opd.kicad_sch
Changed lines of the file:
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@@
 			)
 		)
-		(property "Sheetfile" "untitled.kicad_sch"
+		(property "Sheetfile" "opd.kicad_sch"
 			(at 276.86 196.1646 0)
 			(show_name no)
@@
 			(color 255 229 191 1)
 		)
-		(property "Sheetname" "OPD"
+		(property "Sheetname" "opd"
 			(at 204.47 160.5784 0)
 			(show_name no)

Commit message: loyout and routing
Parts:
- removed TP29: Test-Point, oresat-misc:TestPoint-0.75mm-th, symbol oresat_stuff:Test-Point-0.75mm-th
- added R1: 10m, oresat-passives:1206-B, symbol Device:R_Small_US
- added U9: IP4234CZ6,125, Package_SO:TSOP-6_1.65x3.05mm_P0.95mm, symbol oresat_stuff:ip4234cz6
Connections:
- net GND: now also U9.2 (GND)
- net Power/USB+_IN: no longer names the net of J3.A6 (D+), J3.B6 (D+)
- net Power/USB+_IN: now also U9.1 (CH1)
- net Power/USB-_IN: no longer names the net of J3.A7 (D-), J3.B7 (D-)
- net Power/USB-_IN: now also U9.6 (CH2)
- net Power/VJACK renamed VJACK
- net Power/VUSB_IN renamed VUSB
- net VUSB: now also U9.5 (Vbus)
- net VBUS_CARD renamed current sensing/Vin-
- net current sensing/Vin-: now also R1.2
- net VBUS_HOST renamed VBUS_FLATSAT
- net VBUS_FLATSAT: now also R1.1
- new net opd/USB+: U9.3 (CH1)
- new net opd/USB-: U9.4 (CH2)
Other:
- sheet Power ports: added none; removed USB+, USB+_IN, USB-, USB-_IN, VJACK, VUSB_IN
- sheet current sensing ports: added Vin+, Vin-; removed none
- note added: "current sensing shunt"
- moved on the sheet: C2, J1, J2, J3, J4, R2, R3, TP14, TP15
