File: flatsat-debugger/opd.kicad_sch (KiCad schematic)
At the start: 10 parts, among them U2 INA226

Commit message: loyout and routing
Parts:
- removed R1: 10m, oresat-passives:1206-B, symbol Device:R_Small_US
Connections:
- net VBUS_CARD renamed Vin-
- net VBUS_HOST renamed Vin+
Other:
- note removed: "current sensing"
