File: flatsat-debugger/power.kicad_sch (KiCad schematic)
At the start: 15 parts, among them Q1 DMP2035UQ-7, Q2 DMP2035UQ-7, Q3 DMP2035UQ-7, Q6 31-DMN2053UQ-13CT-ND, SW1 C&K PCM13SMTR, U3 LTC4412xS6, U4 LTC4412xS6, U9 IP4234CZ6,125

Commit message: loyout and routing
Parts:
- removed U9: IP4234CZ6,125, Package_SO:TSOP-6_1.65x3.05mm_P0.95mm, symbol oresat_stuff:ip4234cz6
Connections:
- net VBUS_HOST renamed VBUS_FLATSAT
