File: flatsat-debugger/flatsat-debugger.kicad_pcb (KiCad board)
At the start: 4 copper layers, 50 x 75 mm, 54 parts, among them J1 J-SAMTEC-TFM-120-X1-XXX-D-RA, J2 SFM-120-02-X-DH, J3 USB_C_Receptacle_USB2.0_16P, J4 Barrel_Jack, Q1 DMP2035UQ-7, Q2 DMP2035UQ-7, Q3 DMP2035UQ-7, Q4 DMP2035UQ-7, Q6 31-DMN2053UQ-13CT-ND, SW1 C&K PCM13SMTR, U1 MCP2221AxST, U2 INA226, U3 LTC4412xS6, U4 LTC4412xS6, U5 TS5A21366, U6 MAX892LEUA+T, U7 MIC23050-SYML, U8 LTC4412xS6, U9 IP4234CZ6,125

Commit message: loyout and routing
Parts:
- removed TP29: Test-Point, oresat-misc:TestPoint-0.75mm-th
- added C6: 4.7uF, oresat-passives:0603-A, F.Cu at (154.9, 103.1)
- added D2: AMB, oresat-passives:0603-A, F.Cu at (143.8, 110.7)
- added D3: GRN, oresat-passives:0603-A, F.Cu at (143.8, 113.3)
- added R13: 1k, oresat-passives:0603-A, F.Cu at (147.8, 110.7)
- added R14: 1k, oresat-passives:0603-A, F.Cu at (147.8, 113.3)
- moved R6 106.5 mm to (114.8, 124.5), turned to 180 degrees
- moved R11 105.4 mm to (122.9, 128.0), turned to 90 degrees
- moved TP21 93.3 mm to (125.5, 138.2)
- moved TP20 92.1 mm to (129.0, 138.2)
- moved R19 88.0 mm to (113.3, 98.0), turned to 90 degrees
- moved R18 87.9 mm to (113.3, 94.0), turned to -90 degrees
- moved R17 86.3 mm to (115.3, 98.0), turned to 90 degrees
- moved R16 86.2 mm to (115.3, 94.0), turned to -90 degrees
- moved R20 84.0 mm to (117.3, 94.0), turned to -90 degrees
- moved R21 83.9 mm to (117.3, 98.0), turned to 90 degrees
- moved R22 82.4 mm to (119.4, 94.0), turned to -90 degrees
- moved R23 82.3 mm to (119.4, 98.0), turned to 90 degrees
- moved TP18 80.5 mm to (123.4, 99.1)
- moved SW1 74.4 mm to (117.3, 136.7), turned to 0 degrees
- moved Q6 72.4 mm to (113.8, 128.0), turned to 90 degrees
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Connections:
- net /OPD/LOCAL_SCL renamed /current sensing/LOCAL_SCL
- net /OPD/LOCAL_SDA renamed /current sensing/LOCAL_SDA
- net /OPD/USB+ renamed /opd/USB+
- net /OPD/USB- renamed /opd/USB-
- net /Power/USB+_IN renamed Net-(J3-D+-PadA6)
- net /Power/USB-_IN renamed Net-(J3-D--PadA7)
- net /Power/VJACK renamed VJACK
- net VBUS_CARD renamed /current sensing/Vin-
- net VBUS_HOST renamed VBUS_FLATSAT
- D1 pad 2: /OPD_PWR -> /OPD_SCL
- Q4 pad 3: /OPD_PWR -> /OPD_SCL
- Q6 pad 2: /OPD/USBShutdown -> /Power/USBShutdown
- R6 pad 1: /OPD/USBShutdown -> /Power/USBShutdown
- U1 pad 2: /OPD/USBShutdown -> Net-(D3-A)
- U1 pad 3: unconnected-(U1-GP1-Pad3) -> Net-(D2-A)
- U1 pad 7: unconnected-(U1-GP2-Pad7) -> /Power/USBShutdown
- U5 pad 5: /OPD_SCL -> /OPD_PWR
- U8 pad 6: /OPD_PWR -> /OPD_SCL
Routing:
- net /SPARE21: track 0.00 -> 100.8 mm, vias 0 -> 2
- net /current sensing/LOCAL_SDA: track 0.00 -> 85.4 mm
- net /SPARE31: track 1.60 -> 83.0 mm, vias 1 -> 2
- net /C3-UART-TX: track 0.00 -> 78.1 mm, vias 0 -> 4
- net /C3-UART-RX: track 1.08 -> 70.8 mm, vias 0 -> 2
- net /~{SD}: track 40.8 -> 110.1 mm, vias 0 -> 1
- net /current sensing/LOCAL_SCL: track 0.00 -> 67.6 mm, vias 0 -> 2
- net /Power/USBShutdown: track 0.00 -> 49.7 mm, vias 0 -> 2
- net VUSB: track 9.08 -> 55.3 mm, vias 0 -> 4
- net Net-(Q1-S): track 6.64 -> 52.2 mm, vias 0 -> 4
- net /OPD_SDA: track 68.5 -> 111.2 mm, vias 1 -> 2
- net Net-(U1-GP3): track 0.00 -> 33.8 mm
- net /OPD_PWR: track 68.6 -> 99.8 mm, vias 1 -> 5
- net Net-(Q2-D): track 0.00 -> 29.2 mm, vias 0 -> 2
- net 3.3V: track 0.00 -> 26.0 mm, vias 0 -> 8
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- added copper zone on In1.Cu, net 3.3V
- added copper zone on B.Cu, net GND
- added copper zone on F.Cu, net GND
- added copper zone on In2.Cu, net GND
Other:
- board size 50 x 75 mm -> 75 x 50 mm

Commit message: improved layout
Parts:
- moved R10 1.66 mm to (148.2, 101.6)
- moved C1 0.46 mm to (140.3, 101.6)
- moved C2 0.46 mm to (128.6, 93.0)
- moved C3 0.46 mm to (150.0, 98.6)
- moved C4 0.46 mm to (148.5, 92.5)
- moved C6 0.46 mm to (154.5, 103.1)
- moved D2 0.46 mm to (143.3, 110.7)
- moved D3 0.46 mm to (143.3, 113.3)
- moved J1 0.46 mm to (171.5, 115.2)
- moved J3 0.46 mm to (135.5, 94.3)
- moved J4 0.46 mm to (151.5, 129.6)
- moved L1 0.46 mm to (143.9, 96.5)
- moved Q1 0.46 mm to (130.1, 101.6)
- moved Q2 0.46 mm to (130.1, 128.0)
- moved Q6 0.46 mm to (113.3, 128.0)
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Routing:
- net GND: track 22.7 -> 58.3 mm, vias 2 -> 11
- net /OPD_SCL: track 79.4 -> 107.2 mm, vias 1 -> 3
- net 3.3V: track 26.0 -> 30.1 mm, vias 8 -> 11
- net VBUS_FLATSAT: track 78.7 -> 80.9 mm
- net /~{SD}: track 110.1 -> 111.3 mm
- net /SPARE4: track 69.1 -> 68.3 mm
Other:
- board size 75 x 50 mm -> 76 x 50 mm

Commit message: better layout stuff. ANDREW REVIEW MEEEEE
Parts:
- moved TP20 9.87 mm to (120.5, 132.5)
- moved R14 7.54 mm to (147.0, 105.8), turned to 90 degrees
- moved R13 5.76 mm to (144.5, 105.8), turned to 90 degrees
- moved D3 5.10 mm to (147.0, 109.8), turned to -90 degrees
- moved F2 4.67 mm to (140.5, 133.0), turned to 90 degrees
- moved Q2 3.44 mm to (133.5, 127.5)
- moved TP21 2.63 mm to (126.5, 136.0)
- moved U4 2.13 mm to (125.0, 132.5)
- moved TP14 1.69 mm to (166.0, 112.8)
- moved R11 1.57 mm to (123.0, 129.5), turned to 0 degrees
- moved D2 1.52 mm to (144.5, 109.8), turned to -90 degrees
- moved Q1 0.67 mm to (130.7, 101.9), turned to 0 degrees
Routing:
- net VBUS_FLATSAT: track 80.9 -> 15.8 mm
- net Net-(Q1-S): track 52.2 -> 13.7 mm, vias 4 -> 8
- net /current sensing/LOCAL_SDA: track 85.1 -> 62.3 mm, vias 0 -> 2
- net Net-(Q2-D): track 29.2 -> 12.6 mm
- net /current sensing/Vin-: track 18.2 -> 3.85 mm
- net VJACK: track 14.2 -> 0.00 mm
- net VUSB: track 55.3 -> 42.5 mm, vias 4 -> 2
- net Net-(U4-STAT): track 5.91 -> 13.5 mm
- net /Power/USBShutdown: track 49.7 -> 42.5 mm
- net Net-(Q2-G): track 5.52 -> 12.0 mm, vias 0 -> 2
- net /SPARE21: track 100.8 -> 95.0 mm
- net /OPD_SCL: track 107.2 -> 102.3 mm
- net Net-(D3-A): track 7.55 -> 12.1 mm
- net /OPD_PWR: track 99.3 -> 103.7 mm
- net /SPARE9: track 89.2 -> 85.3 mm
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- added copper zone on F.Cu, net /current sensing/Vin-
- added copper zone on In2.Cu, net 3.3V
- added copper zone on In1.Cu, net GND
- added copper zone on F.Cu, net Net-(Q1-S)
- added copper zone on In2.Cu, net Net-(Q1-S)
- added copper zone on F.Cu, net Net-(Q2-D)
- added copper zone on F.Cu, net VBUS_FLATSAT
- added copper zone on F.Cu, net VJACK
- added copper zone on F.Cu, net VUSB
- removed copper zone on In1.Cu, net 3.3V
- removed copper zone on In2.Cu, net GND
Other:
- board size 76 x 50 mm -> 74.8 x 50 mm
