File: c3-proxy/c3-proxy.kicad_sch (KiCad schematic)
At the start: 19 parts, among them J1 TFM-120-X1-XXX-D-RA, J2 SFM-120-02-L-DH, J3 USB_C_Receptacle_USB2.0_16P, J4 Barrel_Jack_Switch_MountingPin, J5 Conn_01x04, U9 IP4234CZ6,125

Commit message: fixed BOM, silk art scale
Parts:
- C2: DIST (none) -> DigiKey; DPN (none) -> 399-6856-1-ND; MFR (none) -> KEMET; MPN (none) -> C0603C104K5RACAUTO
- J4: DIST (none) -> DigiKey; DPN (none) -> CP-069BPJTR-ND; MFR (none) -> Same Sky (Formerly CUI Devices); MPN (none) -> PJ-069B-SMT-TR
Changed lines of the file:
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@@
 			)
 		)
-		(property "Datasheet" ""
+		(property "Datasheet" "https://www.cuidevices.com/product/resource/pj-069b-smt-tr.pdf"
 			(at 110.49 163.576 0)
 			(hide yes)
@@
 		)
 		(property "Description" "DC Barrel Jack with an internal switch and a mounting pin"
+			(at 109.22 162.56 0)
+			(hide yes)
+			(show_name no)
+			(do_not_autoplace no)
+			(effects
+				(font
+					(size 1.27 1.27)
+				)
+			)
+		)
+		(property "DIST" "DigiKey"
+			(at 109.22 162.56 0)
+			(hide yes)
+			(show_name no)
+			(do_not_autoplace no)
+			(effects
+				(font
+					(size 1.27 1.27)
+				)
+			)
+		)
+		(property "DPN" "CP-069BPJTR-ND"
+			(at 109.22 162.56 0)
+			(hide yes)
+			(show_name no)
+			(do_not_autoplace no)
+			(effects
+				(font
+					(size 1.27 1.27)
+				)
+			)
+		)
+		(property "MFR" "Same Sky (Formerly CUI Devices)"
+			(at 109.22 162.56 0)
+			(hide yes)
+			(show_name no)
+			(do_not_autoplace no)
+			(effects
+				(font
+					(size 1.27 1.27)
+				)
+			)
+		)
+		(property "MPN" "PJ-069B-SMT-TR"
 			(at 109.22 162.56 0)
 			(hide yes)
@@
 			)
 		)
-		(property "Datasheet" ""
+		(property "Datasheet" "https://search.kemet.com/download/specsheet/C0603C104K5RACAUTO"
 			(at 96.52 233.68 0)
 			(hide yes)
@@
 			)
 		)
-		(property "Description" "Unpolarized capacitor, small symbol"
+		(property "Description" "0.1 µF ±10% 50V Ceramic Capacitor X7R 0603 (1608 Metric)"
 			(at 96.52 243.84 0)
 			(hide yes)
 			(show_name no)
+			(do_not_autoplace no)
+			(effects
+				(font
+					(size 1.27 1.27)
+				)
+			)
+		)
+		(property "DIST" "DigiKey"
+			(at 96.52 233.68 0)
+			(hide yes)
+			(show_name no)
+			(do_not_autoplace no)
+			(effects
+				(font
+					(size 1.27 1.27)
+				)
+			)
+		)
+		(property "DPN" "399-6856-1-ND"
+			(at 96.52 233.68 0)
+			(hide yes)
+			(show_name no)
+			(do_not_autoplace no)
+			(effects
+				(font
+					(size 1.27 1.27)
+				)
+			)
+		)
+		(property "MFR" "KEMET"
+			(at 96.52 233.68 0)
+			(hide yes)
+			(show_name no)
+			(do_not_autoplace no)
+			(effects
+				(font
+					(size 1.27 1.27)
+				)
+			)
+		)
+		(property "MPN" "C0603C104K5RACAUTO"
+			(at 96.52 233.68 0)
+			(hide yes)
+			(show_name no)

Commit message: layout cleanup, add bypass to U1-Vdd
Connections:
- net GND: now also J4.MP (MountPin)
- net SPARE1: no longer J1.2, J2.2 (Pin_2)
- new net SPARE2: J1.2, J2.2 (Pin_2)
- no-connect marks 3 -> 2
Other:
- note removed: "not sure the ideal way to connect/route this capacitor"
Changed lines of the file:
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@@
-		)
-	)
-	(text "not sure the ideal way to connect/route this capacitor"
-		(exclude_from_sim no)
-		(at 94.488 246.126 0)
-		(effects
-			(font
-				(size 1.27 1.27)
-			)
 		)
 	)
@@
 	)
 	(junction
-		(at 325.12 38.1)
-		(diameter 0)
-		(color 0 0 0 0)
-	)
-	(junction
 		(at 251.46 76.2)
 		(diameter 0)
@@
 	)
 	(junction
-		(at 158.75 38.1)
-		(diameter 0)
-		(color 0 0 0 0)
-	)
-	(junction
 		(at 158.75 81.28)
 		(diameter 0)
@@
 		(diameter 0)
 		(color 0 0 0 0)
-	)
-	(no_connect
-		(at 109.22 170.18)
 	)
 	(no_connect
@@
 	(wire
 		(pts
+			(xy 109.22 170.18) (xy 109.22 171.45)
+		)
+		(stroke
+			(width 0)
+			(type default)
+		)
+	)
+	(wire
+		(pts
 			(xy 269.24 208.28) (xy 269.24 181.61)
 		)
@@
 	(wire
 		(pts
-			(xy 158.75 40.64) (xy 158.75 38.1)
-		)
-		(stroke
-			(width 0)
-			(type default)
-		)
-	)
-	(wire
-		(pts
 			(xy 154.94 81.28) (xy 158.75 81.28)
 		)
@@
 	(wire
 		(pts
-			(xy 328.93 40.64) (xy 325.12 40.64)
-		)
-		(stroke
-			(width 0)
-			(type default)
-		)
-	)
-	(wire
-		(pts
 			(xy 191.77 208.28) (xy 269.24 208.28)
 		)
@@
 	(wire
 		(pts
-			(xy 325.12 40.64) (xy 325.12 38.1)
-		)
-		(stroke
-			(width 0)
-			(type default)
-		)
-	)
-	(wire
-		(pts
 			(xy 328.93 93.98) (xy 325.12 93.98)
 		)
@@
 	(wire
 		(pts
-			(xy 154.94 40.64) (xy 158.75 40.64)
+			(xy 154.94 40.64) (xy 328.93 40.64)
 		)
 		(stroke
@@
 			)
 			(justify right bottom)
+		)
+	)
+	(label "SPARE2"
+		(at 274.32 40.64 0)
+		(effects
+			(font
+				(size 1.27 1.27)
+			)
+			(justify left bottom)
 		)
 	)
@@
 					(unit 1)
 				)
+			)
+		)
+	)
+	(symbol
+		(lib_id "power:GND")
+		(at 109.22 171.45 0)
+		(unit 1)
+		(body_style 1)
+		(exclude_from_sim no)
+		(in_bom yes)
+		(on_board yes)
+		(in_pos_files yes)
+		(dnp no)
+		(property "Reference" "#PWR030"
+			(at 109.22 177.8 0)
+			(hide yes)
+			(show_name no)
+			(do_not_autoplace no)
+			(effects
+				(font
+					(size 1.27 1.27)
+				)
+			)
+		)
+		(property "Value" "GND"
+			(at 107.188 175.514 0)
+			(show_name no)
+			(do_not_autoplace no)
+			(effects
+				(font
+					(size 1.27 1.27)
+				)
+				(justify left)
+			)
+		)
+		(property "Footprint" ""
+			(at 109.22 171.45 0)
+			(hide yes)
+			(show_name no)
+			(do_not_autoplace no)
+			(effects
+				(font
+					(size 1.27 1.27)
+				)
+			)
+		)
+		(property "Datasheet" ""
+			(at 109.22 171.45 0)
+			(hide yes)
+			(show_name no)
+			(do_not_autoplace no)
+			(effects
+				(font
+					(size 1.27 1.27)
+				)
+			)
+		)
+		(property "Description" "Power symbol creates a global label with name \"GND\" , ground"
+			(at 109.22 171.45 0)
+			(hide yes)
+			(show_name no)
+			(do_not_autoplace no)
+			(effects
+				(font
+					(size 1.27 1.27)
+				)
+			)
+		)
+		(pin "1"
+		)
+		(instances
+			(project "c3-proxy"
+				(path "/1a9202c4-e698-4c93-952c-ee3e64e9e49c"
+					(reference "#PWR030")
+					(unit 1)
+				)

Commit message: Final tweaks on v1.1.
Added more LEDs for main power, polished high power connections, DRC, ERC, etc. Added release folder.
Parts:
- J3: value USB_C_Receptacle_USB2.0_16P -> USB4105-GF-A
- J4: value Barrel_Jack_Switch_MountingPin -> PJ-069B-SMT-TR
- J5: now not fitted
Other:
- note added: "All resistors are 0603 1% unless otherwise noted. All capacitors are 0603 10% X5R Vw >= 25 V unless otherwise noted."
- note added: "External Power (5.5 mm / 2.1 mm Barrel)"
- note added: "USB C"
- note added: "mechanical"
- title: c3-Proxy card -> c3-Proxy Board
- moved on the sheet: C2, FID1, FID2, FID3, HW1, HW2, HW3, J1, J2, J3, J4, R1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
